Commit message: Added laser xacro

File: description/robot_core.xacro (robot description, xacro)
@@ -10,4 +10,7 @@
     <material name="blue">
         <color rgba="0.2 0.2 1 1" />
+    </material>
+     <material name="red">
+        <color rgba="1 0 0 1" />
     </material>
     <material name="black">
