Commit message: Updated params to make odometry more accurate

File: description/robot.urdf.xacro (robot description, xacro)
@@ -4,4 +4,3 @@
     <xacro:include filename="ros2_control.xacro" />
     <xacro:include filename="lidar.xacro" />
-    <xacro:include filename="ros2_control.xacro" />
 </robot>

File: description/robot_core.xacro (robot description, xacro)
@@ -32,5 +32,14 @@
         <color rgba="0 0 0 1" />
     </material>
+    <!-- BASE LINK -->
     <link name="base_link">
+    </link>
+    <!-- BASE FOOTPRINT LINK -->
+    <joint name="base_footprint_joint" type="fixed">
+        <parent link="base_link"/>
+        <child link="base_footprint" />
+        <origin xyz="0 0 0" rpy="0 0 0" />
+    </joint>
+    <link name="base_footprint">
     </link>
     <!-- CHASSIS LINK -->

File: description/ros2_control.xacro (robot description, xacro)
@@ -10,5 +10,6 @@
             <param name="baud_rate">57600</param>
             <param name="timeout">1000</param>
-            <param name="enc_counts_per_rev">1689</param>
+            <param name="enc_counts_per_rev">1684</param>
+            <!-- I actually got 1682, but I am multiplying by 2 because that seems to give me the right result in rviz -->
         </hardware>
         <joint name="left_wheel_joint">
